File: AT28C256 Version/CoCoEPROMpak.kicad_sch (KiCad schematic)
At the start: 8 parts, among them P1 COCO-CART, U1 2732, U2 28C256

Commit message: Added gerber files
Other:
- note added: "4k: * Install 2732 at U1 * JP2, JP3 not used 32k: * Install AT28C256 at U2 * Select 16k bank with JP2"
- note added: "This version with support for EEPROM AT28C256 by RCC@2023 https://github.com/costarc/CoCoEPROMpak"
- note removed: "4k: * Install 2732 at U1 * JP2, JP3 not used 8k: * Install 2764 at U2 * Set JP2 to 1 * Set JP3 to 1 16k: * Install 27128 at U2 * Set JP2 to 1 * Set JP3 to 1 32k: * Install 27256 at U2 * Select 16k bank with JP2 * Set JP3 to 1 64k: * Install 27512 at U2 * Select 16k banks with JP2 and JP3"
Changed lines of the file:
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@@
     (effects (font (size 6.4516 5.4838)) (justify right bottom))
   )
-  (text "4k:\n* Install 2732 at U1\n* JP2, JP3 not used\n8k:\n* Install 2764 at U2\n* Set JP2 to 1\n* Set JP3 to 1\n16k:\n* Install 27128 at U2\n* Set JP2 to 1\n* Set JP3 to 1\n32k:\n* Install 27256 at U2\n* Select 16k bank with JP2\n* Set JP3 to 1\n64k:\n* Install 27512 at U2\n* Select 16k banks with JP2 and JP3"
+  (text "This version with support for EEPROM AT28C256 by RCC@2023\nhttps://github.com/costarc/CoCoEPROMpak"
+    (at 25.4 250.19 180)
+    (effects (font (size 3.81 3.2385)) (justify left bottom))
+  )
+  (text "4k:\n* Install 2732 at U1\n* JP2, JP3 not used\n32k:\n* Install AT28C256 at U2\n* Select 16k bank with JP2"
     (at 27.94 172.72 180)
     (effects (font (size 2.032 2.54)) (justify left bottom))
@@
     (pin "1")
   )
-  (symbol (lib_id "CoCoEPROMpak-eagle-import:ANSI_A") (at 190.5 233.68 0) (unit 2)
-    (in_bom yes) (on_board yes)
-    (property "Reference" "#FRAME1" (id 0) (at 190.5 233.68 0)
-      (effects (font (size 1.27 1.27)) hide)
-    )
-    (property "Value" "ANSI_A" (id 1) (at 190.5 233.68 0)
-      (effects (font (size 1.27 1.27)) hide)
-    )
-    (property "Footprint" "CoCoEPROMpak:" (id 2) (at 190.5 233.68 0)
-      (effects (font (size 1.27 1.27)) hide)
-    )
-    (property "Datasheet" "" (id 3) (at 190.5 233.68 0)
-      (effects (font (size 1.27 1.27)) hide)
-    )
-  )
   (symbol (lib_id "CoCoEPROMpak-eagle-import:+5V_ARROW") (at 195.58 73.66 0) (unit 1)
     (in_bom yes) (on_board yes)
@@
   )
   (symbol_instances
-    (path "/43385896-f10c-414d-8b1a-7f1c61617824"
-      (reference "#FRAME1") (unit 2) (value "ANSI_A") (footprint "CoCoEPROMpak:")
-    )
     (path "/4c82689d-4222-42f4-bf71-f2af47a5ef1f"
       (reference "#U$01") (unit 1) (value "+5V_ARROW") (footprint "CoCoEPROMpak:")

Commit message: Added gerbers with gnd plane added
Parts:
- P1: footprint CoCoEPROMpak:COCO-CART-2.1X1.75 -> Roni Footprints:COCO-CART-2.1X1.75
Changed lines of the file:
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@@
   )
   (text "4k-64k EPROM Cartridge\nfor Tandy/TRS-80 Color Computer"
-    (at 160.02 43.18 180)
+    (at 160.02 43.18 0)
     (effects (font (size 6.4516 5.4838)) (justify right bottom))
   )
   (text "This version with support for EEPROM AT28C256 by RCC@2023\nhttps://github.com/costarc/CoCoEPROMpak"
-    (at 25.4 250.19 180)
+    (at 25.4 250.19 0)
     (effects (font (size 3.81 3.2385)) (justify left bottom))
   )
   (text "4k:\n* Install 2732 at U1\n* JP2, JP3 not used\n32k:\n* Install AT28C256 at U2\n* Select 16k bank with JP2"
-    (at 27.94 172.72 180)
+    (at 27.94 172.72 0)
     (effects (font (size 2.032 2.54)) (justify left bottom))
   )
@@
   )
   (text "CoCoEPROMpak is a free hardware design: you can redistribute it\nand/or modify it under the terms of the GNU General Public License\nas published by the Free Software Foundation, either version 3 of\nthe License, or (at your option) any later version.\nCoCoEPROMpak is distributed in the hope that it will be useful,\nbut WITHOUT ANY WARRANTY; without even the implied warranty\nof MERCHANTABILITY or FITNESS FOR A PARTICULAR PURPOSE.\nSee the GNU General Public License for more details.\nYou should have received a copy of the GNU General Public License\nalong with CoCoEPROMpak. If not, see http://www.gnu.org/licenses/."
-    (at 200.66 193.04 180)
+    (at 200.66 193.04 0)
     (effects (font (size 1.778 1.5113)) (justify left bottom))
   )
@@
   )
   (text "Copyright 2013 by Mark J. Blair\nDistributed under GPLv3\nhttps://github.com/NF6X/CoCoEPROMpak"
-    (at 25.4 228.6 180)
+    (at 25.4 228.6 0)
     (effects (font (size 3.81 3.2385)) (justify left bottom))
   )
@@
       (effects (font (size 1.27 1.27)) hide)
     )
-    (property "Footprint" "CoCoEPROMpak:COCO-CART-2.1X1.75" (id 2) (at 132.08 114.3 0)
+    (property "Footprint" "Roni Footprints:COCO-CART-2.1X1.75" (id 2) (at 132.08 114.3 0)
       (effects (font (size 1.27 1.27)) hide)
     )
@@
     )
     (path "/2b982b89-b771-4ebc-91eb-a0e6cdf221f8"
-      (reference "P1") (unit 1) (value "COCO-CART") (footprint "CoCoEPROMpak:COCO-CART-2.1X1.75")
+      (reference "P1") (unit 1) (value "COCO-CART") (footprint "Roni Footprints:COCO-CART-2.1X1.75")
     )
     (path "/e32794ca-4818-47ba-b086-a599cff1572b"

Commit message: Rev.1
Connections:
- net +5V: now also JP2.3
- net GND: now also JP2.1
- net A14: no longer names the net of P1.38 (A14)
- net A14: no longer JP2.1
- net A15: no longer names the net of P1.39 (A15)
- net A15: no longer JP2.3
- no-connect marks 0 -> 2
Changed lines of the file:
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@@
   (junction (at 177.8 129.54) (diameter 0) (color 0 0 0 0)
   )
+  (junction (at 174.5093 172.5308) (diameter 0) (color 0 0 0 0)
+  )
+  (no_connect (at 147.32 119.38))
+  (no_connect (at 147.32 121.92))
   (bus_entry (at 167.64 116.84) (size -2.54 -2.54)
     (stroke (width 0) (type default) (color 0 0 0 0))
@@
     (stroke (width 0) (type default) (color 0 0 0 0))
   )
+  (wire (pts (xy 174.498 178.562) (xy 174.498 172.5308))
+    (stroke (width 0) (type default) (color 0 0 0 0))
+  )
   (bus (pts (xy 165.1 101.6) (xy 165.1 104.14))
     (stroke (width 0) (type default) (color 0 0 0 0))
@@
     (stroke (width 0) (type default) (color 0 0 0 0))
   )
+  (wire (pts (xy 174.498 172.5308) (xy 174.5093 172.5308))
+    (stroke (width 0) (type default) (color 0 0 0 0))
+  )
   (wire (pts (xy 167.64 116.84) (xy 185.42 116.84))
     (stroke (width 0) (type default) (color 0 0 0 0))
@@
   )
   (wire (pts (xy 152.4 142.24) (xy 152.4 144.78))
+    (stroke (width 0) (type default) (color 0 0 0 0))
+  )
+  (wire (pts (xy 165.1 165.1) (xy 169.418 165.1))
+    (stroke (width 0) (type default) (color 0 0 0 0))
+  )
+  (wire (pts (xy 169.418 165.1) (xy 169.418 178.562))
     (stroke (width 0) (type default) (color 0 0 0 0))
   )
@@
   (label "D0" (at 220.98 83.82 0)
     (effects (font (size 1.2446 1.2446)) (justify left bottom))
-  )
-  (global_label "A15" (shape input) (at 174.498 178.562 90) (fields_autoplaced)
-    (effects (font (size 1 1)) (justify left))
-    (property "Intersheet References" "${INTERSHEET_REFS}" (id 0) (at 174.4355 173.9001 90)
-      (effects (font (size 1 1)) (justify left) hide)
-    )
   )
   (global_label "*WE" (shape input) (at 156.464 177.8 90) (fields_autoplaced)
@@
     )
   )
-  (global_label "A15" (shape input) (at 147.32 121.92 0) (fields_autoplaced)
-    (effects (font (size 1 1)) (justify left))
-    (property "Intersheet References" "${INTERSHEET_REFS}" (id 0) (at 151.9819 121.8575 0)
-      (effects (font (size 1 1)) (justify left) hide)
-    )
-  )
   (global_label "*RW" (shape input) (at 147.32 134.62 0) (fields_autoplaced)
     (effects (font (size 1.27 1.27)) (justify left))
@@
     (effects (font (size 1 1)) (justify left))
     (property "Intersheet References" "${INTERSHEET_REFS}" (id 0) (at 171.8955 169.9477 90)
-      (effects (font (size 1 1)) (justify left) hide)
-    )
-  )
-  (global_label "A14" (shape input) (at 169.418 178.562 90) (fields_autoplaced)
-    (effects (font (size 1 1)) (justify left))
-    (property "Intersheet References" "${INTERSHEET_REFS}" (id 0) (at 169.3555 173.9001 90)
-      (effects (font (size 1 1)) (justify left) hide)
-    )
-  )
-  (global_label "A14" (shape input) (at 147.32 119.38 0) (fields_autoplaced)
-    (effects (font (size 1 1)) (justify left))
-    (property "Intersheet References" "${INTERSHEET_REFS}" (id 0) (at 151.9819 119.3175 0)
       (effects (font (size 1 1)) (justify left) hide)
     )
@@
     (pin "1")
   )
+  (symbol (lib_id "CoCoEPROMpak-eagle-import:+5V_ARROW") (at 174.5093 167.4508 0) (unit 1)
+    (in_bom yes) (on_board yes)
+    (property "Reference" "#U$0101" (id 0) (at 174.5093 167.4508 0)
+      (effects (font (size 1.27 1.27)) hide)
+    )
+    (property "Value" "+5V_ARROW" (id 1) (at 174.5093 167.4508 0)
+      (effects (font (size 1.27 1.27)) hide)
+    )
+    (property "Footprint" "CoCoEPROMpak:" (id 2) (at 174.5093 167.4508 0)
+      (effects (font (size 1.27 1.27)) hide)
+    )
+    (property "Datasheet" "" (id 3) (at 174.5093 167.4508 0)
+      (effects (font (size 1.27 1.27)) hide)
+    )
+    (pin "1")
+  )
   (symbol (lib_id "CoCoEPROMpak-eagle-import:+5V_ARROW") (at 195.58 73.66 0) (unit 1)
     (in_bom yes) (on_board yes)
@@
     (pin "1")
   )
+  (symbol (lib_id "CoCoEPROMpak-eagle-import:GND") (at 165.1 167.64 0) (unit 1)
+    (in_bom yes) (on_board yes)
+    (property "Reference" "#U$0102" (id 0) (at 165.1 167.64 0)
+      (effects (font (size 1.27 1.27)) hide)
+    )
+    (property "Value" "GND" (id 1) (at 165.1 167.64 0)
+      (effects (font (size 1.27 1.27)) hide)
+    )
+    (property "Footprint" "CoCoEPROMpak:" (id 2) (at 165.1 167.64 0)
+      (effects (font (size 1.27 1.27)) hide)
+    )
+    (property "Datasheet" "" (id 3) (at 165.1 167.64 0)
+      (effects (font (size 1.27 1.27)) hide)
+    )
+    (pin "1")
+  )
   (symbol (lib_id "CoCoEPROMpak-eagle-import:C-US050-025X075") (at 86.36 101.6 0) (unit 1)
     (in_bom yes) (on_board yes)
@@
       (reference "#U$09") (unit 1) (value "+5V_ARROW") (footprint "CoCoEPROMpak:")
     )
+    (path "/3fd4a117-0c51-4edc-b583-1a69718e14c1"
+      (reference "#U$0101") (unit 1) (value "+5V_ARROW") (footprint "CoCoEPROMpak:")
+    )
+    (path "/a912e45f-8585-4ea9-838e-02d9d0304f8c"
+      (reference "#U$0102") (unit 1) (value "GND") (footprint "CoCoEPROMpak:")
+    )
     (path "/ae864cb5-2dc1-42c2-aa42-4a864c2be714"
